Commit message: Correccio posicio lidar i red piece

File: src/my_robot_description/urdf/rubot/rubot_mecanum_custom.urdf (robot description, URDF)
Before this commit: robot rubot, 10 links, 9 joints
Joints:
- joint red_piece_joint: origin xyz=-0.1 0.01 0.06 rpy=0 0 0 -> xyz=0.10 0.0 0.08 rpy=0 0 0
- joint scan_joint: origin xyz=0 0 0.14 rpy=0 0 0 -> xyz=0 0 0.14 rpy=0 0 3.14
